File: Teensy Board.brd (EAGLE design)
At the start: 2 parts

Commit message: changes in Teensy Breakout Board
Parts:
- removed SV4: (no value), con-lstb:MA12-1
- added SV1: (no value), con-lstb:MA13-1
Connections:
- removed net AGND: U$1.AGND
- net N$1: now also SV1.2, SV1.3, U$1.AGND, U$1.GND; no longer SV4.1, U$1.3.3V
- net N$10: now also SV1.6, U$1.5; no longer SV4.6, U$1.6
- net N$11: now also SV1.5, U$1.4; no longer SV4.5, U$1.5
- net N$12: now also SV1.4, U$1.14/A0; no longer SV4.4, U$1.4
- net N$2: now also SV1.1, U$1.3.3V; no longer SV4.2, U$1.GND
- net N$3: now also SV1.13, U$1.12; no longer SV4.3, U$1.14/A0
- net N$4: now also SV1.12, U$1.11; no longer SV4.12, U$1.12
- net N$5: now also SV1.11, U$1.10; no longer SV4.11, U$1.11
- net N$6: now also SV1.10, U$1.9; no longer SV4.10, U$1.10
- net N$7: now also SV1.9, U$1.8; no longer SV4.9, U$1.9
- net N$8: now also SV1.8, U$1.7; no longer SV4.8, U$1.8
- net N$9: now also SV1.7, U$1.6; no longer SV4.7, U$1.7
Routing:
- net N$3: track 32.6 -> 6.35 mm
- net N$12: track 6.35 -> 32.6 mm
- net N$2: track 10.3 -> 22.6 mm
- net N$1: track 33.9 -> 27.3 mm
Changed lines of the file:
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@@
 <elements>
 <element name="U$1" library="Teensy_3_and_LC_Series_Boards_v1.4" package="TEENSY_3.0-3.2&amp;LC_DIL+4" value="TEENSY_3.1-3.2_DIL+4" x="24.13" y="53.34"/>
-<element name="SV4" library="con-lstb" package="MA12-1" value="" x="10.16" y="50.8" rot="R270">
-<attribute name="MPN" value="" x="10.16" y="50.8" size="0.8128" layer="27" rot="R270" display="off"/>
-<attribute name="OC_NEWARK" value="unknown" x="10.16" y="50.8" size="0.8128" layer="27" rot="R270" display="off"/>
-<attribute name="OC_FARNELL" value="unknown" x="10.16" y="50.8" size="0.8128" layer="27" rot="R270" display="off"/>
-<attribute name="MF" value="" x="10.16" y="50.8" size="0.8128" layer="27" rot="R270" display="off"/>
+<element name="SV1" library="con-lstb" package="MA13-1" value="" x="10.16" y="52.07" rot="R270">
+<attribute name="MF" value="" x="10.16" y="52.07" size="1.778" layer="27" rot="R270" display="off"/>
+<attribute name="OC_NEWARK" value="unknown" x="10.16" y="52.07" size="1.778" layer="27" rot="R270" display="off"/>
+<attribute name="MPN" value="" x="10.16" y="52.07" size="1.778" layer="27" rot="R270" display="off"/>
+<attribute name="OC_FARNELL" value="unknown" x="10.16" y="52.07" size="1.778" layer="27" rot="R270" display="off"/>
 </element>
 </elements>
 <signals>
-<signal name="AGND">
-<contactref element="U$1" pad="AGND"/>
-</signal>
 <signal name="VIN">
 <contactref element="U$1" pad="VIN"/>
@@
 <contactref element="U$1" pad="VUSB"/>
 </signal>
+<signal name="N$1">
+<contactref element="U$1" pad="GND"/>
+<contactref element="U$1" pad="AGND"/>
+<contactref element="SV1" pad="2"/>
+<contactref element="SV1" pad="3"/>
+<wire x1="11.43" y1="64.77" x2="16.51" y2="69.85" width="0.254" layer="16"/>
+<wire x1="10.16" y1="64.77" x2="11.43" y2="64.77" width="0.254" layer="16"/>
+<wire x1="29.21" y1="69.85" x2="31.75" y2="67.31" width="0.254" layer="1"/>
+<wire x1="16.51" y1="69.85" x2="29.21" y2="69.85" width="0.254" layer="1"/>
+<wire x1="10.16" y1="64.77" x2="10.16" y2="62.23" width="0.254" layer="1"/>
+</signal>
+<signal name="N$2">
+<contactref element="U$1" pad="3.3V"/>
+<contactref element="SV1" pad="1"/>
+<wire x1="30.7975" y1="65.7225" x2="31.75" y2="64.77" width="0.254" layer="1"/>
+<wire x1="17.145" y1="65.7225" x2="30.7975" y2="65.7225" width="0.254" layer="1"/>
+<wire x1="16.8275" y1="66.04" x2="17.145" y2="65.7225" width="0.254" layer="1"/>
+<wire x1="12.7" y1="66.04" x2="16.8275" y2="66.04" width="0.254" layer="1"/>
+<wire x1="11.43" y1="67.31" x2="12.7" y2="66.04" width="0.254" layer="1"/>
+<wire x1="10.16" y1="67.31" x2="11.43" y2="67.31" width="0.254" layer="1"/>
+</signal>
+<signal name="N$3">
+<contactref element="SV1" pad="13"/>
+<contactref element="U$1" pad="12"/>
+<wire x1="10.16" y1="36.83" x2="16.51" y2="36.83" width="0.254" layer="1"/>
+</signal>
+<signal name="N$4">
+<contactref element="SV1" pad="12"/>
+<contactref element="U$1" pad="11"/>
+<wire x1="10.16" y1="39.37" x2="16.51" y2="39.37" width="0.254" layer="16"/>
+</signal>
+<signal name="N$5">
+<contactref element="SV1" pad="11"/>
+<contactref element="U$1" pad="10"/>
+<wire x1="10.16" y1="41.91" x2="16.51" y2="41.91" width="0.254" layer="1"/>
+</signal>
+<signal name="N$6">
+<contactref element="SV1" pad="10"/>
+<contactref element="U$1" pad="9"/>
+<wire x1="10.16" y1="44.45" x2="16.51" y2="44.45" width="0.254" layer="1"/>
+</signal>
+<signal name="N$7">
+<contactref element="SV1" pad="9"/>
+<contactref element="U$1" pad="8"/>
+<wire x1="10.16" y1="46.99" x2="16.51" y2="46.99" width="0.254" layer="1"/>
+</signal>
+<signal name="N$8">
+<contactref element="SV1" pad="8"/>
+<contactref element="U$1" pad="7"/>
+<wire x1="10.16" y1="49.53" x2="16.51" y2="49.53" width="0.254" layer="1"/>
+</signal>
+<signal name="N$9">
+<contactref element="SV1" pad="7"/>
+<contactref element="U$1" pad="6"/>
+<wire x1="10.16" y1="52.07" x2="16.51" y2="52.07" width="0.254" layer="1"/>
+</signal>
+<signal name="N$10">
+<contactref element="SV1" pad="6"/>
+<contactref element="U$1" pad="5"/>
+<wire x1="10.16" y1="54.61" x2="16.51" y2="54.61" width="0.254" layer="1"/>
+</signal>
+<signal name="N$11">
+<contactref element="SV1" pad="5"/>
+<contactref element="U$1" pad="4"/>
+<wire x1="10.16" y1="57.15" x2="16.51" y2="57.15" width="0.254" layer="1"/>
+</signal>
+<signal name="N$12">
+<contactref element="SV1" pad="4"/>
+<contactref element="U$1" pad="14/A0"/>
+<wire x1="17.78" y1="53.34" x2="31.75" y2="39.37" width="0.254" layer="16"/>
+<wire x1="12.7" y1="53.34" x2="17.78" y2="53.34" width="0.254" layer="16"/>
+<wire x1="12.7" y1="57.785" x2="12.7" y2="53.34" width="0.254" layer="16"/>
+<wire x1="10.795" y1="59.69" x2="12.7" y2="57.785" width="0.254" layer="16"/>
+<wire x1="10.16" y1="59.69" x2="10.795" y2="59.69" width="0.254" layer="16"/>
+</signal>
 <signal name="N$13">
 <polygon width="0.4064" layer="1">
@@
 </polygon>
 </signal>
-<signal name="N$1">
-<contactref element="U$1" pad="3.3V"/>
-<contactref element="SV4" pad="1"/>
-<wire x1="17.78" y1="64.77" x2="31.75" y2="64.77" width="0.254" layer="16"/>
-<wire x1="17.78" y1="70.485" x2="17.78" y2="64.77" width="0.254" layer="16"/>
-<wire x1="17.145" y1="71.12" x2="17.78" y2="70.485" width="0.254" layer="16"/>
-<wire x1="10.16" y1="71.12" x2="17.145" y2="71.12" width="0.254" layer="16"/>
-<wire x1="10.16" y1="64.77" x2="10.16" y2="71.12" width="0.254" layer="16"/>
-</signal>
-<signal name="N$2">
-<contactref element="SV4" pad="2"/>
-<contactref element="U$1" pad="GND"/>
-<wire x1="12.065" y1="65.405" x2="16.51" y2="69.85" width="0.254" layer="16"/>
-<wire x1="12.065" y1="64.135" x2="12.065" y2="65.405" width="0.254" layer="16"/>
-<wire x1="10.16" y1="62.23" x2="12.065" y2="64.135" width="0.254" layer="16"/>
-</signal>
-<signal name="N$3">
-<contactref element="SV4" pad="3"/>
-<contactref element="U$1" pad="14/A0"/>
-<wire x1="17.78" y1="53.34" x2="31.75" y2="39.37" width="0.254" layer="16"/>
-<wire x1="12.065" y1="53.34" x2="17.78" y2="53.34" width="0.254" layer="16"/>
-<wire x1="12.065" y1="57.785" x2="12.065" y2="53.34" width="0.254" layer="16"/>
-<wire x1="10.16" y1="59.69" x2="12.065" y2="57.785" width="0.254" layer="16"/>
-</signal>
-<signal name="N$4">
-<contactref element="SV4" pad="12"/>
-<contactref element="U$1" pad="12"/>
-<wire x1="10.16" y1="36.83" x2="16.51" y2="36.83" width="0.254" layer="16"/>
-</signal>
-<signal name="N$5">
-<contactref element="SV4" pad="11"/>
-<contactref element="U$1" pad="11"/>
-<wire x1="10.16" y1="39.37" x2="16.51" y2="39.37" width="0.254" layer="16"/>
-</signal>
-<signal name="N$6">
-<contactref element="SV4" pad="10"/>
-<contactref element="U$1" pad="10"/>
-<wire x1="10.16" y1="41.91" x2="16.51" y2="41.91" width="0.254" layer="16"/>
-</signal>
-<signal name="N$7">
-<contactref element="SV4" pad="9"/>
-<contactref element="U$1" pad="9"/>
-<wire x1="10.16" y1="44.45" x2="16.51" y2="44.45" width="0.254" layer="16"/>
-</signal>
-<signal name="N$8">
-<contactref element="SV4" pad="8"/>
-<contactref element="U$1" pad="8"/>
-<wire x1="10.16" y1="46.99" x2="16.51" y2="46.99" width="0.254" layer="16"/>
-</signal>
-<signal name="N$9">
-<contactref element="SV4" pad="7"/>
-<contactref element="U$1" pad="7"/>
-<wire x1="10.16" y1="49.53" x2="16.51" y2="49.53" width="0.254" layer="16"/>
-</signal>
-<signal name="N$10">
-<contactref element="SV4" pad="6"/>
-<contactref element="U$1" pad="6"/>
-<wire x1="10.16" y1="52.07" x2="16.51" y2="52.07" width="0.254" layer="16"/>
-</signal>
-<signal name="N$11">
-<contactref element="SV4" pad="5"/>
-<contactref element="U$1" pad="5"/>
-<wire x1="10.16" y1="54.61" x2="16.51" y2="54.61" width="0.254" layer="1"/>
-</signal>
-<signal name="N$12">
-<contactref element="SV4" pad="4"/>
-<contactref element="U$1" pad="4"/>
-<wire x1="10.16" y1="57.15" x2="16.51" y2="57.15" width="0.254" layer="1"/>
-</signal>
 <signal name="N$14">
